File: Schaltplan.brd (EAGLE design)
At the start: 14 parts, among them IC1 ICL7665CSA, Q2 IRF4905

Commit message: v 1.2
Parts:
- removed R23: 20 kΩ, eagle-ltspice:R1206
- added BATTERY, OUTPUT: (no value), con-wago-500:W237-102
- added D1: 1N4004, diode:DO41-10
- added F1: (no value), fuse:GSH15
- added LED3: red (low current), led:KA-3528ASYC
- added R1, R2: 5,6 kΩ, eagle-ltspice:R1206
- added U$1: PIN-GENERIC, 0liver:LEER
- C1: value (none) -> 100nF
- LED1: value green -> green (low current)
- LED2: value red -> yellow (low current); device led:SML0603 -> led:KA-3528ASYC
- R11: value 130 kΩ -> 120 kΩ
- moved C1 69.1 mm to (-3.68, -17.5)
- moved R21 38.9 mm to (27.1, 6.57), turned to 0 degrees
- moved R22 29.4 mm to (30.9, 8.86), turned to 180 degrees
- moved R3 28.4 mm to (32.7, 20.8), turned to 270 degrees
- moved R13 23.0 mm to (24.8, 21.5), turned to 0 degrees
- moved IC1 21.7 mm to (23.4, 16.7)
- moved R12 14.9 mm to (19.3, 21.6), turned to 0 degrees
- moved R11 14.4 mm to (17.1, 15.4)
- moved R42 13.2 mm to (37.7, 15.7)
- moved LED2 11.2 mm to (42.4, 19.5), turned to 90 degrees
- moved LED1 10.7 mm to (39.7, 19.5), turned to 90 degrees
- moved Q2 9.79 mm to (28.1, 9.95), turned to 90 degrees
- moved R41 7.35 mm to (35.9, 20.8), turned to 90 degrees
Connections:
- removed net OUT-POWER: Q2.D, R41.2
- new net N$10: R42.2
- new net N$17: R1.2, R11.1
- new net N$18: BATTERY.1, F1.1
- new net N$4: OUTPUT.2, Q2.D, R41.2
- net GND: now also BATTERY.2, D1.A, LED3.C, OUTPUT.1, R1.1; no longer R11.1
- net N$1: now also LED3.A, R2.1; no longer IC1.5, R22.2, R23.1
- net N$5: no longer R42.2
- net POWER: now also D1.C, F1.2, R2.2, R22.2; no longer R23.2
Routing:
- net GND: track 0.38 -> 56.4 mm, vias 1 -> 0
- net N$7: track 23.6 -> 57.0 mm
- net N$4: track 0.00 -> 32.6 mm
- net OUT-POWER: track 28.9 -> 0.00 mm, vias 1 -> 0
- net N$5: track 30.2 -> 11.3 mm
- net N$10: track 0.00 -> 11.7 mm
- net N$1: track 10.6 -> 0.00 mm
- net N$2: track 11.4 -> 18.9 mm
- net N$16: track 4.97 -> 0.00 mm
- net POWER: track 57.2 -> 52.6 mm, vias 1 -> 0
- net N$3: track 11.2 -> 9.06 mm
- net N$6: track 11.7 -> 9.93 mm
- added copper zone on layer 1, net N$11
- added copper zone on layer 1, net N$12
- added copper zone on layer 16, net N$13
- added copper zone on layer 1, net N$14
- added copper zone on layer 16, net N$15
- added copper zone on layer 16, net N$4
- added copper zone on layer 16, net N$7
- added copper zone on layer 16, net POWER
- added copper zone on layer 16, net S$1
Other:
- board outline added: 55.5 x 26.2 mm
- board text added: "12.2014"
- board text added: "FULL"
- board text added: "V1.2"
- board text added: "www.tief-dunkel-kalt.org"
- board text removed: "01.2015"
- board text removed: "< 80%"
- board text removed: "V1.3"
- board text removed: "tief-dunkel-kalt.org"
