File: Tiefenentladeschutz 2.sch (EAGLE design)
At the start: 37 parts, among them IC1 ICL7665CSA, IC2 NE555D, T2 BCV26 PNP

Commit message: v2.4
Parts:
- removed R1, R9: 100k, eagle-ltspice:RR1206
- removed T2: BCV26 PNP, transistor:-PNP-SOT23-BCE
- added T1: (no value), transistor:BC817-40-NPN-SOT23-BEC
Connections:
- new net N$26: 1.1, 8.1, C1.1, F1.2, IC1.V+, R2.2, R5.2, R7.2, T1.C
- net GND: no longer T2.C
- net N$1: now also R10.2; no longer R1.1, R2.2
- net N$10: no longer R10.2
- net N$22: no longer T2.E
- net N$7: now also T1.B; no longer R9.2, T2.B
- net V+: now also T1.E; no longer 1.1, 8.1, C1.1, F1.2, IC1.V+, R1.2, R5.2, R7.2, R9.1
Other:
- moved on the sheet: C5, R10, R15, R17

Commit message: 2.6
Parts:
- removed T1, T3, T4: (no value), transistor:BC817-40-NPN-SOT23-BEC
- added D1: 1N4004, diode:1N4004
- added R1: 0, eagle-ltspice:RR1206
- added R18: 5,6k, eagle-ltspice:RR1206
- added R9: 100k, eagle-ltspice:RR1206
- added U$2: IRLML9301, 0liver:IRLML9301
- added U$3, U$4: IRLML6346, 0liver:IRLML6346
- C4: value 10 nF -> 10nF; device eagle-ltspice:CC1206 -> rcl:C-EUC0805K
- F1: value FUSESH22,5A -> 0,5A
- R13: value 30k -> 8,2k
- R14: value 510 -> 680
- R3: value 130k -> 120k
- R4: value ? -> 470k
- R8: value ? -> 4,7k
Connections:
- net GND: now also D1.A, R18.1, U$2.D; no longer R3.1
- net N$1: now also R1.1, R2.2; no longer R10.2
- net N$10: now also R10.2
- net N$17: now also U$3.G; no longer T4.B
- net N$18: now also U$4.G; no longer T3.B
- net N$21: now also U$4.D; no longer T3.C
- net N$22: now also U$2.S, U$4.S; no longer T3.E
- net N$26: now also R18.2, R3.1; no longer 1.1, 8.1, C1.1, F1.2, IC1.V+, R2.2, R5.2, R7.2, T1.C
- net N$3: now also U$3.S; no longer T4.E
- net N$7: now also R9.2, U$2.G; no longer T1.B
- net V+: now also 1.1, 8.1, C1.1, D1.C, F1.2, IC1.V+, R1.2, R5.2, R7.2, R9.1, U$3.D; no longer T1.E, T4.C
Other:
- moved on the sheet: R10, R15, R17, R3

Commit message: 2.7
Parts:
- removed LED3: blue, led:LEDP-LCC-2
- removed R11: 200k, 0liver:POTENTIOMETER
- added LED5: OSTAR_4-LEWE2B-MXPX-6K8L, led:OSTAR_4-LEWE2B-MXPX-6K8L
- SUMMER: value SUMMER -> SUMMER3; device 0liver:SUMMER -> 0liver:SUMMER3
Connections:
- removed net N$14: R11.2, R12.2
- removed net N$22: C2.2, C3.2, C4.2, IC2.GND, LED3.C, R15.2, R17.2, SUMMER.-, U$2.S, U$4.S
- new net 2NDGND: C2.2, C3.2, C4.2, IC2.GND, LED5.C, R15.2, R17.2, SUMMER.-, U$2.S, U$4.S
- net N$12: now also LED5.A; no longer LED3.A
- net V+: now also R12.2; no longer R11.1, R11.3
Other:
- moved on the sheet: R16
Changed lines of the file:
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@@
 <part name="R14" library="eagle-ltspice" deviceset="R" device="R1206" value="680"/>
 <part name="R10" library="eagle-ltspice" deviceset="R" device="R1206" value="6,8 k"/>
-<part name="R11" library="0liver" deviceset="POTENTIOMETER" device="" value="200k"/>
-<part name="SUMMER" library="0liver" deviceset="SUMMER" device=""/>
-<part name="LED3" library="led" deviceset="LED" device="P-LCC-2" value="blue"/>
+<part name="SUMMER" library="0liver" deviceset="SUMMER" device="3" value="SUMMER3"/>
 <part name="X1" library="con-ptr500" deviceset="AK300/2" device=""/>
 <part name="R16" library="resistor" deviceset="R-EU_" device="0617/17" value="27 "/>
@@
 <part name="D1" library="diode" deviceset="1N4004" device=""/>
 <part name="C4" library="rcl" deviceset="C-EU" device="C0805K" value="10nF"/>
+<part name="LED5" library="led" deviceset="OSTAR_4-" device="LEWE2B-MXPX-6K8L"/>
 </parts>
 <sheets>
@@
 <instance part="R14" gate="G$1" x="154.94" y="76.2" rot="R180"/>
 <instance part="R10" gate="G$1" x="68.58" y="35.56" rot="R180"/>
-<instance part="R11" gate="R$1" x="144.78" y="88.9" rot="R90"/>
 <instance part="SUMMER" gate="G$1" x="86.36" y="58.42"/>
-<instance part="LED3" gate="G$1" x="190.5" y="27.94"/>
 <instance part="X1" gate="-1" x="-53.34" y="58.42"/>
 <instance part="X1" gate="-2" x="-53.34" y="53.34"/>
-<instance part="R16" gate="G$1" x="190.5" y="45.72" rot="R90"/>
+<instance part="R16" gate="G$1" x="190.5" y="60.96" rot="R90"/>
 <instance part="1" gate="G$1" x="-30.48" y="71.12" rot="R270"/>
 <instance part="LED4" gate="G$1" x="-30.48" y="48.26"/>
@@
 <instance part="D1" gate="1" x="-35.56" y="55.88" rot="R90"/>
 <instance part="C4" gate="G$1" x="99.06" y="53.34"/>
+<instance part="LED5" gate="G$1" x="190.5" y="40.64"/>
 </instances>
 <busses>
@@
 <pinref part="IC2" gate="A" pin="V+"/>
 <wire x1="127" y1="60.96" x2="132.08" y2="60.96" width="0.1524" layer="91"/>
-<wire x1="132.08" y1="60.96" x2="132.08" y2="88.9" width="0.1524" layer="91"/>
+<wire x1="132.08" y1="60.96" x2="132.08" y2="96.52" width="0.1524" layer="91"/>
 <pinref part="C2" gate="G$1" pin="1"/>
-<wire x1="132.08" y1="88.9" x2="132.08" y2="96.52" width="0.1524" layer="91"/>
 <wire x1="124.46" y1="43.18" x2="132.08" y2="43.18" width="0.1524" layer="91"/>
 <wire x1="132.08" y1="60.96" x2="132.08" y2="43.18" width="0.1524" layer="91"/>
@@
 <wire x1="88.9" y1="96.52" x2="93.98" y2="96.52" width="0.1524" layer="91"/>
 <junction x="132.08" y="96.52"/>
-<junction x="132.08" y="88.9"/>
 <junction x="144.78" y="96.52"/>
-<wire x1="141.16" y1="88.9" x2="132.08" y2="88.9" width="0.1524" layer="91"/>
 <wire x1="-30.48" y1="96.52" x2="-30.48" y2="76.2" width="0.1524" layer="91"/>
 <junction x="-30.48" y="96.52"/>
@@
 <junction x="-20.32" y="96.52"/>
 <junction x="50.8" y="96.52"/>
-<pinref part="R11" gate="R$1" pin="1"/>
-<pinref part="R11" gate="R$1" pin="3"/>
 <pinref part="SUMMER" gate="G$1" pin="+"/>
 <junction x="86.36" y="96.52"/>
@@
 <wire x1="-35.56" y1="96.52" x2="-35.56" y2="58.42" width="0.1524" layer="91"/>
 <junction x="-35.56" y="96.52"/>
+<pinref part="R12" gate="G$1" pin="2"/>
+<wire x1="144.78" y1="96.52" x2="144.78" y2="73.66" width="0.1524" layer="91"/>
 </segment>
 </net>
@@
 </segment>
 </net>
-<net name="N$14" class="0">
-<segment>
-<pinref part="R12" gate="G$1" pin="2"/>
-<wire x1="144.78" y1="73.66" x2="144.78" y2="83.44" width="0.1524" layer="91"/>
-<pinref part="R11" gate="R$1" pin="2"/>
-</segment>
-</net>
 <net name="N$19" class="0">
 <segment>
@@
 <net name="N$12" class="0">
 <segment>
-<pinref part="LED3" gate="G$1" pin="A"/>
-<wire x1="190.5" y1="40.64" x2="190.5" y2="30.48" width="0.1524" layer="91"/>
+<wire x1="190.5" y1="55.88" x2="190.5" y2="48.26" width="0.1524" layer="91"/>
 <pinref part="R16" gate="G$1" pin="1"/>
+<pinref part="LED5" gate="G$1" pin="A"/>
 </segment>
 </net>
@@
 </segment>
 </net>
-<net name="N$22" class="0">
-<segment>
-<pinref part="LED3" gate="G$1" pin="C"/>
+<net name="2NDGND" class="0">
+<segment>
 <wire x1="86.36" y1="52.07" x2="86.36" y2="43.18" width="0.1524" layer="91"/>
-<wire x1="190.5" y1="22.86" x2="190.5" y2="17.78" width="0.1524" layer="91"/>
 <pinref part="C3" gate="G$1" pin="2"/>
+<wire x1="190.5" y1="25.4" x2="190.5" y2="17.78" width="0.1524" layer="91"/>
 <wire x1="144.78" y1="20.32" x2="144.78" y2="17.78" width="0.1524" layer="91"/>
 <junction x="144.78" y="17.78"/>
@@
 <junction x="106.68" y="27.94"/>
 <pinref part="C4" gate="G$1" pin="2"/>
+<pinref part="LED5" gate="G$1" pin="C"/>
 </segment>
 </net>
@@
 <pinref part="U$3" gate="G$1" pin="S"/>
 <pinref part="R16" gate="G$1" pin="2"/>
-<wire x1="190.5" y1="78.74" x2="190.5" y2="50.8" width="0.1524" layer="91"/>
-</segment>
-</net>
+<wire x1="190.5" y1="78.74" x2="190.5" y2="66.04" width="0.1524" layer="91"/>
+</segment>
+</net>

Commit message: 3.0
Parts:
- removed C5: 470 uF, rcl:CPOL-EUTT5D10
- removed D1: 1N4004, diode:1N4004
- removed F1: 0,5A, fuse:FUSESH22,5A
- removed LED5: OSTAR_4-LEWE2B-MXPX-6K8L, led:OSTAR_4-LEWE2B-MXPX-6K8L
- removed R(B): 0 ohm, eagle-ltspice:RR1206
- removed R17: 1k, eagle-ltspice:RR1206
- removed SUMMER: SUMMER3, 0liver:SUMMER3
- removed X1: (no value), con-ptr500:AK300/2
- added LED3: (no value), led:LEDP-LCC-2
- added Q1: NMOSFET-D2PAK-7, D2pak-7:NMOSFET-D2PAK-7
- added R11: 68k, eagle-ltspice:RR1206
- added U$6: IRLML9301, 0liver:IRLML9301
- added X3: (no value), con-ptr500:AK500/3
- C1: device eagle-ltspice:CC0603 -> eagle-ltspice:CC1206
- LED1: value red 2mA -> green 2mA
- LED2: value green 2mA -> red 2mA
- R1: value 0 -> 100k
- R10: value 6,8 k -> 68k
- R15, R9: value 100k -> 470k
- R16: device resistor:R-EU_0617/17 -> resistor:R-EU_0414/15
Connections:
- removed net N$23: C5.+, R17.1
- removed net POWER-IN: F1.1, X1-1.KL
- new net N$13: IC1.HYST1, R1.1, R2.2
- new net N$16: IC1.OUT1, LED1.C, R10.2
- new net N$22: Q1.G, R11.1, R15.1
- net 2NDGND: now also LED3.C; no longer LED5.C, R15.2, R17.2, SUMMER.-
- net GND: now also Q1.S1, Q1.S2, Q1.S3, Q1.S4, Q1.S5, R15.2, X3-3.KL; no longer C5.-, D1.A, R15.1, X1-2.KL
- net N$1: now also Q1.D, X3-2.KL; no longer IC1.HYST2, R1.1, R2.2
- net N$10: now also R11.2, U$6.D; no longer IC1.OUT2, LED1.C, R10.2
- net N$11: now also IC1.OUT2; no longer IC1.OUT1
- net N$12: now also LED3.A; no longer LED5.A
- net N$2: now also IC1.SET1; no longer IC1.SET2
- net N$4: now also IC1.SET2; no longer IC1.SET1
- net N$7: now also U$6.G
- net V+: now also U$6.S, X3-1.KL; no longer D1.C, F1.2, SUMMER.+
Other:
- note added: "+"
- note added: "-"
- note added: "6-14V"
- note added: "GND Last"
- note added: "Optional"
- note removed: "Brücken für einseitiges Layout:"
- moved on the sheet: C2, C3, C4, IC2, R10, R12, R13, R14, R15, R16, R4, R8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

Commit message: 3.3
Parts:
- removed 1: 5,6k, eagle-ltspice:RR1206
- removed C2: 100 nF, eagle-ltspice:CC0603
- removed C3: 10 µF, eagle-ltspice:CC1206
- removed C4: 10nF, rcl:C-EUC0805K
- removed IC2: NE555D, linear:NE555D
- removed LED3: (no value), led:LEDP-LCC-2
- removed LED4: yellow 2mA, eagle-ltspice:LED_ESML0603
- removed R12: 42,2k, eagle-ltspice:RR1206
- removed R13: 8,2k, eagle-ltspice:RR1206
- removed R14: 680, eagle-ltspice:RR1206
- removed R16: 27, resistor:R-EU_0414/15
- removed R8: 4,7k, eagle-ltspice:RR1206
- removed U$2: IRLML9301, 0liver:IRLML9301
- removed U$3, U$4: IRLML6346, 0liver:IRLML6346
- added U$7: IRLML6346, 0liver:IRLML6346
- R4: value 470k -> 0
Connections:
- removed net 2NDGND: C2.2, C3.2, C4.2, IC2.GND, LED3.C, U$2.S, U$4.S
- removed net N$12: LED3.A, R16.1
- removed net N$15: IC2.DIS, R12.1, R13.2
- removed net N$17: R8.2, U$3.G
- removed net N$18: R14.1, U$4.G
- removed net N$19: C4.1, IC2.CV
- removed net N$20: C3.1, IC2.THR, IC2.TR, R13.1
- removed net N$21: R4.2, R8.1, U$4.D
- removed net N$8: IC2.Q, R14.2
- removed net N$9: 1.2, LED4.A
- new net N$23: IC1.OUT2, R4.1
- net GND: no longer LED4.C, U$2.D
- net N$11: now also U$7.D; no longer IC1.OUT2
- net N$22: now also U$7.G
- net N$3: now also R4.2, U$7.S; no longer R16.2, U$3.S
- net N$7: no longer U$2.G
- net V+: no longer 1.1, C2.1, IC2.R, IC2.V+, R12.2, R4.1, U$3.D
Other:
- note removed: "Optional"
- moved on the sheet: 8, LED1, LED2, Q1, R10, R11, R15, R4, R7, R9, U$6, X3-2

Commit message: 3.5
Parts:
- removed 8, R18: 5,6k, eagle-ltspice:RR1206
- removed R15: 470k, eagle-ltspice:RR1206
- removed U$6: IRLML9301, 0liver:IRLML9301
- removed U$7: IRLML6346, 0liver:IRLML6346
- added R12: 100k, eagle-ltspice:RR1206
- added R13: 0, eagle-ltspice:RR1206
- added R8: 470k, eagle-ltspice:RR1206
- added U$2: IRLML9301, 0liver:IRLML9301
- added U$3: IRLML6346, 0liver:IRLML6346
- R1: value 100k -> 820k
- R11: value 68k -> 5,6k
- R2: value 750k -> 100k
- R3: value 120k -> 100k
- R4: value 0 -> 750k
- R5: value 820k -> 120k
- R6: value 100k -> 5,6k
- R9: value 470k -> 68k
Connections:
- removed net N$10: R11.2, U$6.D
- new net N$8: R9.1, U$2.S
- net GND: now also R12.2, R2.1; no longer R15.2, R18.1
- net N$11: now also U$3.D; no longer U$7.D
- net N$13: now also R3.1, R4.2; no longer R1.1, R2.2
- net N$2: now also R4.1, R5.2; no longer R2.1, R3.2
- net N$22: now also R12.1, U$2.D, U$3.G; no longer R11.1, R15.1, U$7.G
- net N$23: now also R13.1; no longer R4.1
- net N$26: now also R5.1, R6.2; no longer R18.2, R3.1
- net N$3: now also R13.2, U$3.S; no longer R4.2, U$7.S
- net N$4: now also R1.1, R2.2; no longer R5.1, R6.2
- net N$5: now also R11.2; no longer 8.2
- net N$7: now also R8.2, U$2.G; no longer R9.2, U$6.G
- net V+: now also R11.1, R3.2, R8.1, R9.2; no longer 8.1, R5.2, R9.1, U$6.S
Other:
- note added: "GND OUT"
- note removed: "6-14V"
- note removed: "GND Last"
- moved on the sheet: LED1, Q1, R1, R10, R11, R2, R3, R4, R5, R6, R7, R9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

Commit message: 3.7
Parts:
- removed R13: 0, eagle-ltspice:RR1206
- removed X3: (no value), con-ptr500:AK500/3
- added RB: 0, eagle-ltspice:RR1206
- added U$4: (no value), 0liver:PINBIG
- added U$6, U$7: (no value), 0liver:PIN1.27
- renumbered Q1 to Q4
Connections:
- removed net N$23: IC1.OUT2, R13.1
- new net N$10: R9.2, RB.1
- net GND: now also U$6.P$1; no longer X3-3.KL
- net N$1: now also U$7.P$1; no longer X3-2.KL
- net N$3: now also IC1.OUT2; no longer R13.2
- net V+: now also RB.2, U$4.P$1; no longer R9.2, X3-1.KL
Other:
- note removed: "-"
