File: Tiefenentladeschutz-ohneLed.brd (EAGLE design)
At the start: 30 x 37 mm, 15 parts, among them IC1 ICL7665CSA, Q4 NMOSFET-D2PAK-7, T1 BC856B

Commit message: R12 to 100kOhm
Parts:
- R12: value 20k -> 100k
Changed lines of the file:
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@@
 <attribute name="SPICEPREFIX" value="R" x="17.2" y="16.9" size="1.778" layer="27" rot="R90" display="off"/>
 </element>
-<element name="R12" library="eagle-ltspice" package="R1206" value="20k" x="13.02" y="26.66" rot="R180">
+<element name="R12" library="eagle-ltspice" package="R1206" value="100k" x="13.02" y="26.66" rot="R180">
 <attribute name="SPICEMODEL" value="NONE" x="13.02" y="26.66" size="1.778" layer="27" rot="R180" display="off"/>
 <attribute name="SPICEPREFIX" value="R" x="13.02" y="26.66" size="1.778" layer="27" rot="R180" display="off"/>
